Commit message: fucked up urdf trying to fix rotation

File: src/audix_pkg/urdf/audix.urdf (robot description, URDF)
Before this commit: robot audix, 30 links, 29 joints
Joints:
- joint back_left_wheel_joint: origin xyz=-0.0700000000053768 -0.307389999999987 0.024999999990612 rpy=1.57079632679489 0 0 -> xyz=0.0886599999946232 -0.156599999999987 0.024999999990612 rpy=1.57079632679489 0 0
- joint back_right_wheel_joint: origin xyz=-0.0700000000053771 0.00739000000001488 0.0249999999906142 rpy=1.57079632679489 0 0 -> xyz=0.0886599999946229 0.15818000000001488 0.0249999999906142 rpy=1.57079632679489 0 0
- joint front_left_wheel_joint: origin xyz=-0.250000000005374 -0.307389999999985 0.024999999989585 rpy=1.57079632679489 0 0 -> xyz=-0.091340000005374 -0.156599999999985 0.024999999989585 rpy=1.57079632679489 0 0
- joint front_right_wheel_joint: origin xyz=-0.250000000005375 0.00739000000001477 0.0249999999895845 rpy=1.57079632679489 0 0 -> xyz=-0.091340000005375 0.15818000000001477 0.0249999999895845 rpy=1.57079632679489 0 0
- joint imu_joint: origin xyz=-0.15866 -0.15079 0.010 rpy=0 0 0 -> xyz=0 0 0.010 rpy=0 0 0
- joint ir_back_joint: origin xyz=0.00389 -0.15402 0.01325 rpy=0 1.5707963267949 0 -> xyz=0.16255 -0.00323 0.01325 rpy=0 1.5707963267949 0
- joint ir_front_joint: origin xyz=-0.36061 -0.14597 0.01325 rpy=0 1.5707963267949 3.1415926535898 -> xyz=-0.20195 0.00482 0.01325 rpy=0 1.5707963267949 3.1415926535898
- joint ir_front_left_joint: origin xyz=-0.34189 -0.27041 0.01325 rpy=0 1.5707963267949 -2.3561944901923 -> xyz=-0.18323 -0.11962 0.01325 rpy=0 1.5707963267949 -2.3561944901923
- joint ir_front_right_joint: origin xyz=-0.33619 -0.02391 0.01325 rpy=0 1.5707963267949 2.3561944901923 -> xyz=-0.17753 0.12688 0.01325 rpy=0 1.5707963267949 2.3561944901923
- joint ir_left_joint: origin xyz=-0.16403 -0.30425 0.01325 rpy=0 1.5707963267949 -1.5707963267949 -> xyz=-0.00537 -0.15346 0.01325 rpy=0 1.5707963267949 -1.5707963267949
- joint ir_right_joint: origin xyz=-0.15593 0.00425 0.01325 rpy=0 1.5707963267949 1.5707963267949 -> xyz=0.00273 0.15504 0.01325 rpy=0 1.5707963267949 1.5707963267949
- joint scissors_lift_base_fix: origin xyz=-0.310000000005584 -0.150000000000003 0.0124999999899842 rpy=0 0 0 -> xyz=-0.151340000005584 0.0007900000000009999 0.0124999999899842 rpy=0 0 0

Commit message: ts might be peak

File: src/audix_pkg/urdf/audix.urdf (robot description, URDF)
Before this commit: robot audix, 30 links, 29 joints
Links:
- link base_link: geometry visual mesh filename=package://audix/meshes/base_link.STL
